File: PmodUsbUlpi.sch (KiCad schematic (older format))
At the start: 18 parts, among them J1 USB_C_Receptacle_USB2.0, J2 PMOD1, J3 PMOD2, U1 TPS76318, U2 USB3320

Commit message: First Version with Waveshare Pinout
Parts:
- removed J2: PMOD1, Connector_PinHeader_2.54mm:PinHeader_2x06_P2.54mm_Horizontal, symbol Connector_Generic:Conn_02x06_Odd_Even
- removed J3: PMOD2, Connector_PinHeader_2.54mm:PinHeader_2x06_P2.54mm_Horizontal, symbol Connector_Generic:Conn_02x06_Odd_Even
- added J2: 2x10 Header, Connector_PinHeader_2.54mm:PinHeader_2x10_P2.54mm_Horizontal, symbol Connector_Generic:Conn_02x10_Odd_Even
- J1: symbol Connector:USB_C_Receptacle_USB2.0 -> PmodUsbUlpi-rescue:USB_C_Receptacle_USB2.0-Connector
- U2: symbol twam-Misc:USB3320 -> PmodUsbUlpi-rescue:USB3320-twam-Misc
Connections:
- wire segments 115 -> 109
- no-connect marks 9 -> 7
Other:
- note removed: "GND"
- note removed: "IO1"
- note removed: "IO2"
- note removed: "IO3"
- note removed: "IO4"
- note removed: "IO5"
- note removed: "IO6"
- note removed: "IO7"
- note removed: "IO8"
- note removed: "VCC"
